File: pcb/Sensor inputs.kicad_sch (KiCad schematic)
At the start: 3 parts, among them J3 Screw_Terminal_01x03, J4 Screw_Terminal_01x03, J5 Screw_Terminal_01x02

Commit message: redesigning the circuit of the rellay and starting to adjust the footprints
Parts:
- removed J4: Screw_Terminal_01x03, symbol Connector:Screw_Terminal_01x03
- added J10: Screw_Terminal_01x03, TerminalBlock_Phoenix:TerminalBlock_Phoenix_MKDS-1,5-3_1x03_P5.00mm_Horizontal, symbol Connector:Screw_Terminal_01x03
- added J4: Screw_Terminal_01x04, symbol Connector:Screw_Terminal_01x04
- J3: footprint (none) -> TerminalBlock_Phoenix:TerminalBlock_Phoenix_MKDS-1,5-3_1x03_P5.00mm_Horizontal; amazon link (none) -> https://www.amazon.com/QSYZAIL-Screw-Terminal-Circuit-Conne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
- J5: footprint (none) -> TerminalBlock_Phoenix:TerminalBlock_Phoenix_MKDS-1,5-2_1x02_P5.00mm_Horizontal; amazon link (none) -> https://www.amazon.com/QSYZAIL-Screw-Terminal-Circuit-Conne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
Connections:
- net +3.3V: now also J10.3 (Pin_3), J4.4 (Pin_4)
- net GND: now also J10.1 (Pin_1), J4.1 (Pin_1)
- net light sensor: now also J4.3 (Pin_3)
- new net air sensor: J4.2 (Pin_2)
- new net soil_temp: J10.2 (Pin_2)
Other:
- note added: "light and air sensor input"
- note added: "soil tempature input"
- note removed: "light sensor"

Commit message: finishing the bom and adding the jlc number of the parts
Parts:
- J10, J3: jlc part # (none) -> C8270
- J4: footprint (none) -> TerminalBlock_Phoenix:TerminalBlock_Phoenix_MKDS-1,5-4_1x04_P5.00mm_Horizontal; jlc part # (none) -> C90087
- J5: jlc part # (none) -> C3703
Changed lines of the file:
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@@
+			)
+		)
+		(property "jlc part #" "C8270"
+			(at 143.51 76.2 0)
+			(effects
+				(font
+					(size 1.27 1.27)
+				)
+				(hide yes)
 			)
 		)
@@
 			)
 		)
+		(property "jlc part #" "C3703"
+			(at 142.24 129.54 0)
+			(effects
+				(font
+					(size 1.27 1.27)
+				)
+				(hide yes)
+			)
+		)
 		(pin "2"
 		)
@@
 			)
 		)
-		(property "Footprint" ""
+		(property "Footprint" "TerminalBlock_Phoenix:TerminalBlock_Phoenix_MKDS-1,5-4_1x04_P5.00mm_Horizontal"
 			(at 142.24 104.14 0)
 			(effects
@@
 			)
 		)
+		(property "jlc part #" "C90087"
+			(at 142.24 104.14 0)
+			(effects
+				(font
+					(size 1.27 1.27)
+				)
+				(hide yes)
+			)
+		)
 		(pin "2"
 		)
@@
 			(at 142.24 154.94 0)
 			(effects
+				(font
+					(size 1.27 1.27)
+				)
+				(hide yes)
+			)
+		)
+		(property "jlc part #" "C8270"
+			(at 142.24 154.94 0)
+			(effects

Commit message: Finishing the carrier board with the new usb-c modul
Parts:
- renumbered J4 to J2, J5 to J3, J10 to J4, J3 to J5
Changed lines of the file:
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@@
 		(dnp no)
 		(fields_autoplaced yes)
-		(property "Reference" "J3"
+		(property "Reference" "J5"
 			(at 143.51 67.31 0)
 			(show_name no)
@@
 			(project "pcb"
 				(path "/2955ee96-3683-4cf6-bfa3-83b5e4980920/fb52141c-2646-4aaf-afae-845bb8079ac4"
-					(reference "J3")
+					(reference "J5")
 					(unit 1)
 				)
@@
 		(dnp no)
 		(fields_autoplaced yes)
-		(property "Reference" "#PWR012"
+		(property "Reference" "#PWR08"
 			(at 143.51 127 0)
 			(hide yes)
@@
 			(project "pcb"
 				(path "/2955ee96-3683-4cf6-bfa3-83b5e4980920/fb52141c-2646-4aaf-afae-845bb8079ac4"
-					(reference "#PWR012")
+					(reference "#PWR08")
 					(unit 1)
 				)
@@
 		(dnp no)
 		(fields_autoplaced yes)
-		(property "Reference" "#PWR014"
+		(property "Reference" "#PWR09"
 			(at 143.51 152.4 0)
 			(hide yes)
@@
 			(project "pcb"
 				(path "/2955ee96-3683-4cf6-bfa3-83b5e4980920/fb52141c-2646-4aaf-afae-845bb8079ac4"
-					(reference "#PWR014")
+					(reference "#PWR09")
 					(unit 1)
 				)
@@
 		(dnp no)
 		(fields_autoplaced yes)
-		(property "Reference" "#PWR011"
+		(property "Reference" "#PWR07"
 			(at 153.67 106.68 0)
 			(hide yes)
@@
 			(project "pcb"
 				(path "/2955ee96-3683-4cf6-bfa3-83b5e4980920/fb52141c-2646-4aaf-afae-845bb8079ac4"
-					(reference "#PWR011")
+					(reference "#PWR07")
 					(unit 1)
 				)
@@
 		(dnp no)
 		(fields_autoplaced yes)
-		(property "Reference" "J5"
+		(property "Reference" "J3"
 			(at 142.24 120.65 0)
 			(show_name no)
@@
 			(project "pcb"
 				(path "/2955ee96-3683-4cf6-bfa3-83b5e4980920/fb52141c-2646-4aaf-afae-845bb8079ac4"
-					(reference "J5")
+					(reference "J3")
 					(unit 1)
 				)
@@
 		(dnp no)
 		(fields_autoplaced yes)
-		(property "Reference" "#PWR017"
+		(property "Reference" "#PWR010"
 			(at 153.67 157.48 0)
 			(hide yes)
@@
 			(project "pcb"
 				(path "/2955ee96-3683-4cf6-bfa3-83b5e4980920/fb52141c-2646-4aaf-afae-845bb8079ac4"
-					(reference "#PWR017")
+					(reference "#PWR010")
 					(unit 1)
 				)
@@
 		(dnp no)
 		(fields_autoplaced yes)
-		(property "Reference" "J4"
+		(property "Reference" "J2"
 			(at 142.24 92.71 0)
 			(show_name no)
@@
 			(project "pcb"
 				(path "/2955ee96-3683-4cf6-bfa3-83b5e4980920/fb52141c-2646-4aaf-afae-845bb8079ac4"
-					(reference "J4")
+					(reference "J2")
 					(unit 1)
 				)
@@
 		(dnp no)
 		(fields_autoplaced yes)
-		(property "Reference" "#PWR010"
+		(property "Reference" "#PWR013"
 			(at 144.78 99.06 0)
 			(hide yes)
@@
 			(project "pcb"
 				(path "/2955ee96-3683-4cf6-bfa3-83b5e4980920/fb52141c-2646-4aaf-afae-845bb8079ac4"
-					(reference "#PWR010")
+					(reference "#PWR013")
 					(unit 1)
 				)
@@
 		(dnp no)
 		(fields_autoplaced yes)
-		(property "Reference" "#PWR09"
+		(property "Reference" "#PWR012"
 			(at 154.94 78.74 0)
 			(hide yes)
@@
 			(project "pcb"
 				(path "/2955ee96-3683-4cf6-bfa3-83b5e4980920/fb52141c-2646-4aaf-afae-845bb8079ac4"
-					(reference "#PWR09")
+					(reference "#PWR012")
 					(unit 1)
 				)
@@
 		(dnp no)
 		(fields_autoplaced yes)
-		(property "Reference" "J10"
+		(property "Reference" "J4"
 			(at 142.24 146.05 0)
 			(show_name no)
@@
 			(project "pcb"
 				(path "/2955ee96-3683-4cf6-bfa3-83b5e4980920/fb52141c-2646-4aaf-afae-845bb8079ac4"
-					(reference "J10")
+					(reference "J4")
 					(unit 1)
 				)
@@
 		(dnp no)
 		(fields_autoplaced yes)
-		(property "Reference" "#PWR08"
+		(property "Reference" "#PWR011"
 			(at 144.78 73.66 0)
 			(hide yes)
@@
 			(project "pcb"
 				(path "/2955ee96-3683-4cf6-bfa3-83b5e4980920/fb52141c-2646-4aaf-afae-845bb8079ac4"
-					(reference "#PWR08")
-					(unit 1)
-				)
+					(reference "#PWR011")
+					(unit 1)
+				)
