File: pcb/control.kicad_sch (KiCad schematic)
At the start: 3 parts, among them J11 Conn_01x02_Pin

Commit message: Finishing the usb-c module
Parts:
- J11: jlc part # (none) -> C37208
Changed lines of the file:
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@@
 			)
 		)
-		(property "jlc part #" ""
+		(property "jlc part #" "C37208"
 			(at 119.38 102.87 0)
 			(hide yes)
