File: pcb/led_control.kicad_sch (KiCad schematic)
At the start: 4 parts, among them J9 Screw_Terminal_01x02, Q2 AO3400A

Commit message: redesigning the circuit of the rellay and starting to adjust the footprints
Parts:
- J9: footprint (none) -> TerminalBlock_Phoenix:TerminalBlock_Phoenix_MKDS-1,5-2_1x02_P5.00mm_Horizontal; amazon link (none) -> https://www.amazon.com/QSYZAIL-Screw-Terminal-Circuit-Conne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
Changed lines of the file:
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@@
+			)
+		)
+		(property "amazon link" ""
+			(at 153.67 107.95 0)
+			(effects
+				(font
+					(size 1.27 1.27)
+				)
+				(hide yes)
 			)
 		)
@@
 			)
 		)
-		(property "Footprint" ""
+		(property "Footprint" "TerminalBlock_Phoenix:TerminalBlock_Phoenix_MKDS-1,5-2_1x02_P5.00mm_Horizontal"
 			(at 156.21 93.98 0)
 			(effects
@@
 		(property "Description" "Generic screw terminal, single row, 01x02, script generated (kicad-library-utils/schlib/autogen/connector/)"
 			(at 156.21 93.98 0)
+			(effects
+				(font
+					(size 1.27 1.27)
+				)
+				(hide yes)
+			)
+		)
+		(property "amazon link" "https://www.amazon.com/QSYZAIL-Screw-Terminal-Circuit-Connector/dp/B0G4MYNHBC/132-4224079-3597343"
+			(at 156.21 93.98 90)
 			(effects
 				(font
@@
 			)
 		)
+		(property "amazon link" ""
+			(at 140.97 107.95 90)
+			(effects
+				(font
+					(size 1.27 1.27)
+				)
+				(hide yes)
+			)
+		)
 		(pin "1"
 		)
@@
 			(at 144.78 111.76 0)
 			(effects
+				(font
+					(size 1.27 1.27)
+				)
+				(hide yes)
+			)
+		)
+		(property "amazon link" ""
+			(at 144.78 111.76 0)
+			(effects

Commit message: finishing the bom and adding the jlc number of the parts
Parts:
- J9: jlc part # (none) -> C3703
- Q2: amazon link (none) -> https://www.amazon.com/100Pcs-AO3400A-SOT-23-5-8A-N-Channel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; jlc part # (none) -> C20917
- R3: footprint (none) -> Resistor_SMD:R_0603_1608Metric_Pad0.98x0.95mm_HandSolder; amazon link (none) -> https://www.amazon.com/Chanzon-Resistor-Tolerance-Resistors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; jlc part # (none) -> C23179
- R4: footprint (none) -> Resistor_SMD:R_0603_1608Metric_Pad0.98x0.95mm_HandSolder; amazon link (none) -> https://www.amazon.com/100PCS-0603-SMD-chip-resistors/dp/B0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; jlc part # (none) -> C15401
Changed lines of the file:
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@@
 			)
 		)
-		(property "amazon link" ""
+		(property "amazon link" "https://www.amazon.com/100Pcs-AO3400A-SOT-23-5-8A-N-Channel/dp/B0FJ1HTN1Y"
+			(at 153.67 107.95 0)
+			(effects
+				(font
+					(size 1.27 1.27)
+				)
+				(hide yes)
+			)
+		)
+		(property "jlc part #" "C20917"
 			(at 153.67 107.95 0)
 			(effects
@@
 			)
 		)
+		(property "jlc part #" "C3703"
+			(at 156.21 93.98 90)
+			(effects
+				(font
+					(size 1.27 1.27)
+				)
+				(hide yes)
+			)
+		)
 		(pin "2"
 		)
@@
 			)
 		)
-		(property "Footprint" ""
+		(property "Footprint" "Resistor_SMD:R_0603_1608Metric_Pad0.98x0.95mm_HandSolder"
 			(at 140.97 106.172 90)
 			(effects
@@
 			)
 		)
-		(property "amazon link" ""
+		(property "amazon link" "https://www.amazon.com/Chanzon-Resistor-Tolerance-Resistors-Certificated/dp/B08R8CC8RG"
+			(at 140.97 107.95 90)
+			(effects
+				(font
+					(size 1.27 1.27)
+				)
+				(hide yes)
+			)
+		)
+		(property "jlc part #" "C23179"
 			(at 140.97 107.95 90)
 			(effects
@@
 			)
 		)
-		(property "Footprint" ""
+		(property "Footprint" "Resistor_SMD:R_0603_1608Metric_Pad0.98x0.95mm_HandSolder"
 			(at 143.002 111.76 90)
 			(effects
@@
 			)
 		)
-		(property "amazon link" ""
+		(property "amazon link" "https://www.amazon.com/100PCS-0603-SMD-chip-resistors/dp/B0B3SY4DCP?"
 			(at 144.78 111.76 0)
 			(effects
+				(font
+					(size 1.27 1.27)
+				)
+				(hide yes)
+			)
+		)
+		(property "jlc part #" "C15401"
+			(at 144.78 111.76 0)
+			(effects

Commit message: fixing the layout
Parts:
- R4: amazon link https://www.amazon.com/100PCS-0603-SMD-chip-resistors/dp/B0B3SY4DCP? -> https://www.amazon.com/100PCS-0603-SMD-chip-resistors/dp/B0B3SY4DCP? https://www.amazon.com/100PCS-0603-SMD-chip-resistors/dp/B0B3SY4DCP?; jlc part # C15401 -> C2906982
Changed lines of the file:
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@@
 			)
 		)
-		(property "amazon link" "https://www.amazon.com/100PCS-0603-SMD-chip-resistors/dp/B0B3SY4DCP?"
+		(property "amazon link" "https://www.amazon.com/100PCS-0603-SMD-chip-resistors/dp/B0B3SY4DCP? https://www.amazon.com/100PCS-0603-SMD-chip-resistors/dp/B0B3SY4DCP?"
 			(at 144.78 111.76 0)
 			(effects
@@
 			)
 		)
-		(property "jlc part #" "C15401"
+		(property "jlc part #" "C2906982"
 			(at 144.78 111.76 0)
 			(effects

Commit message: separating the pcb components from the other BOM
Parts:
- J9: amazon link https://www.amazon.com/QSYZAIL-Screw-Terminal-Circuit-Conne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 -> (none)
- Q2: amazon link https://www.amazon.com/100Pcs-AO3400A-SOT-23-5-8A-N-Channel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 -> (none)
- R3: amazon link https://www.amazon.com/Chanzon-Resistor-Tolerance-Resistors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 -> (none)
- R4: amazon link https://www.amazon.com/100PCS-0603-SMD-chip-resistors/dp/B0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 -> (none)
Changed lines of the file:
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@@
-			)
-		)
-		(property "amazon link" "https://www.amazon.com/100Pcs-AO3400A-SOT-23-5-8A-N-Channel/dp/B0FJ1HTN1Y"
-			(at 153.67 107.95 0)
-			(effects
-				(font
-					(size 1.27 1.27)
-				)
-				(hide yes)
 			)
 		)
@@
 			)
 		)
-		(property "amazon link" "https://www.amazon.com/QSYZAIL-Screw-Terminal-Circuit-Connector/dp/B0G4MYNHBC/132-4224079-3597343"
-			(at 156.21 93.98 90)
-			(effects
-				(font
-					(size 1.27 1.27)
-				)
-				(hide yes)
-			)
-		)
 		(property "jlc part #" "C3703"
 			(at 156.21 93.98 90)
@@
 			)
 		)
-		(property "amazon link" "https://www.amazon.com/Chanzon-Resistor-Tolerance-Resistors-Certificated/dp/B08R8CC8RG"
-			(at 140.97 107.95 90)
-			(effects
-				(font
-					(size 1.27 1.27)
-				)
-				(hide yes)
-			)
-		)
 		(property "jlc part #" "C23179"
 			(at 140.97 107.95 90)
@@
 			(at 144.78 111.76 0)
 			(effects
-				(font
-					(size 1.27 1.27)
-				)
-				(hide yes)
-			)
-		)
-		(property "amazon link" "https://www.amazon.com/100PCS-0603-SMD-chip-resistors/dp/B0B3SY4DCP? https://www.amazon.com/100PCS-0603-SMD-chip-resistors/dp/B0B3SY4DCP?"
-			(at 144.78 111.76 0)
-			(effects
