File: pcb/led_control.kicad_sch (KiCad schematic)
At the start: 4 parts, among them J9 Screw_Terminal_01x02, Q2 AO3400A

Commit message: Finishing the carrier board with the new usb-c modul
Parts:
- renumbered J9 to J7, Q2 to Q1, R3 to R1, R4 to R2
Changed lines of the file:
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@@
 		(in_pos_files yes)
 		(dnp no)
-		(property "Reference" "#PWR021"
+		(property "Reference" "#PWR018"
 			(at 161.29 105.41 0)
 			(hide yes)
@@
 			(project "pcb"
 				(path "/2955ee96-3683-4cf6-bfa3-83b5e4980920/89a50dcd-3e40-47dd-9489-bea03b3b4f69"
-					(reference "#PWR021")
+					(reference "#PWR018")
 					(unit 1)
 				)
@@
 		(dnp no)
 		(fields_autoplaced yes)
-		(property "Reference" "Q2"
+		(property "Reference" "Q1"
 			(at 160.02 106.6799 0)
 			(show_name no)
@@
 			(project "pcb"
 				(path "/2955ee96-3683-4cf6-bfa3-83b5e4980920/89a50dcd-3e40-47dd-9489-bea03b3b4f69"
-					(reference "Q2")
+					(reference "Q1")
 					(unit 1)
 				)
@@
 		(dnp no)
 		(fields_autoplaced yes)
-		(property "Reference" "#PWR020"
+		(property "Reference" "#PWR017"
 			(at 156.21 121.92 0)
 			(hide yes)
@@
 			(project "pcb"
 				(path "/2955ee96-3683-4cf6-bfa3-83b5e4980920/89a50dcd-3e40-47dd-9489-bea03b3b4f69"
-					(reference "#PWR020")
+					(reference "#PWR017")
 					(unit 1)
 				)
@@
 		(in_pos_files yes)
 		(dnp no)
-		(property "Reference" "J9"
+		(property "Reference" "J7"
 			(at 156.21 89.408 90)
 			(show_name no)
@@
 			(project "pcb"
 				(path "/2955ee96-3683-4cf6-bfa3-83b5e4980920/89a50dcd-3e40-47dd-9489-bea03b3b4f69"
-					(reference "J9")
+					(reference "J7")
 					(unit 1)
 				)
@@
 		(dnp no)
 		(fields_autoplaced yes)
-		(property "Reference" "#PWR019"
+		(property "Reference" "#PWR016"
 			(at 144.78 121.92 0)
 			(hide yes)
@@
 			(project "pcb"
 				(path "/2955ee96-3683-4cf6-bfa3-83b5e4980920/89a50dcd-3e40-47dd-9489-bea03b3b4f69"
-					(reference "#PWR019")
+					(reference "#PWR016")
 					(unit 1)
 				)
@@
 		(dnp no)
 		(fields_autoplaced yes)
-		(property "Reference" "R3"
+		(property "Reference" "R1"
 			(at 140.97 101.6 90)
 			(show_name no)
@@
 			(project "pcb"
 				(path "/2955ee96-3683-4cf6-bfa3-83b5e4980920/89a50dcd-3e40-47dd-9489-bea03b3b4f69"
-					(reference "R3")
+					(reference "R1")
 					(unit 1)
 				)
@@
 		(dnp no)
 		(fields_autoplaced yes)
-		(property "Reference" "R4"
+		(property "Reference" "R2"
 			(at 147.32 110.4899 0)
 			(show_name no)
@@
 			(project "pcb"
 				(path "/2955ee96-3683-4cf6-bfa3-83b5e4980920/89a50dcd-3e40-47dd-9489-bea03b3b4f69"
-					(reference "R4")
+					(reference "R2")
 					(unit 1)
 				)
