File: pcb/light_sensor.kicad_sch (KiCad schematic)
At the start: 4 parts, among them J7 Screw_Terminal_01x04, U3 AM2302

Commit message: separating the pcb components from the other BOM
Parts:
- J7: amazon link https://www.amazon.com/QSYZAIL-Screw-Terminal-Circuit-Conne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 -> (none)
- R1: amazon link https://www.amazon.com/100PCS-0603-SMD-chip-resistors/dp/B0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 -> (none)
- R2: amazon link https://www.amazon.com/eBoot-Photoresistor-Sensitive-Resist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 -> (none)
Changed lines of the file:
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@@
-			)
-		)
-		(property "amazon link" ""
-			(at 104.14 124.46 0)
-			(effects
-				(font
-					(size 1.27 1.27)
-				)
-				(hide yes)
 			)
 		)
@@
 			)
 		)
-		(property "amazon link" "https://www.amazon.com/eBoot-Photoresistor-Sensitive-Resistor-Dependent/dp/B01N7V536K?"
-			(at 114.3 96.52 0)
-			(effects
-				(font
-					(size 1.27 1.27)
-				)
-				(hide yes)
-			)
-		)
 		(property "jlc part #" "C10077"
 			(at 114.3 96.52 0)
@@
 			)
 		)
-		(property "amazon link" "https://www.amazon.com/100PCS-0603-SMD-chip-resistors/dp/B0B3SY4DCP? https://www.amazon.com/100PCS-0603-SMD-chip-resistors/dp/B0B3SY4DCP?"
-			(at 114.3 104.14 0)
-			(effects
-				(font
-					(size 1.27 1.27)
-				)
-				(hide yes)
-			)
-		)
 		(property "jlc part #" "C2906982"
 			(at 114.3 104.14 0)
@@
 			(at 67.31 109.22 0)
 			(effects
-				(font
-					(size 1.27 1.27)
-				)
-				(hide yes)
-			)
-		)
-		(property "amazon link" "https://www.amazon.com/QSYZAIL-Screw-Terminal-Circuit-Connector/dp/B0G4MYNHBC/132-4224079-3597343"
-			(at 67.31 109.22 0)
-			(effects
