File: pcb/power.kicad_sch (KiCad schematic)
At the start: 6 parts, among them J1 Screw_Terminal_01x02, U1 AMS1117-3.3

Commit message: redesigning the circuit of the rellay and starting to adjust the footprints
Parts:
- C1, C3: footprint (none) -> Resistor_SMD:R_0603_1608Metric_Pad0.98x0.95mm_HandSolder
- C2, C4: footprint (none) -> Capacitor_THT:CP_Radial_D5.0mm_P2.50mm
- J1: footprint (none) -> TerminalBlock_Phoenix:TerminalBlock_Phoenix_MKDS-1,5-2_1x02_P5.00mm_Horizontal; amazon link (none) -> https://www.amazon.com/QSYZAIL-Screw-Terminal-Circuit-Conne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
Connections:
- net +5V: now reaches C1.1, C2.1, J1.2 (Pin_2), U1.3 (VI)
Changed lines of the file:
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@@
+	)
+	(junction
+		(at 142.24 96.52)
+		(diameter 0)
+		(color 0 0 0 0)
 	)
 	(junction
@@
 	(wire
 		(pts
-			(xy 135.89 96.52) (xy 144.78 96.52)
+			(xy 135.89 96.52) (xy 142.24 96.52)
 		)
 		(stroke
@@
 	(wire
 		(pts
+			(xy 142.24 96.52) (xy 144.78 96.52)
+		)
+		(stroke
+			(width 0)
+			(type default)
+		)
+	)
+	(wire
+		(pts
 			(xy 119.38 96.52) (xy 135.89 96.52)
 		)
@@
 			(width 0)
 			(type default)
+		)
+	)
+	(symbol
+		(lib_id "power:+5V")
+		(at 142.24 96.52 0)
+		(unit 1)
+		(exclude_from_sim no)
+		(in_bom yes)
+		(on_board yes)
+		(dnp no)
+		(fields_autoplaced yes)
+		(property "Reference" "#PWR027"
+			(at 142.24 100.33 0)
+			(effects
+				(font
+					(size 1.27 1.27)
+				)
+				(hide yes)
+			)
+		)
+		(property "Value" "+5V"
+			(at 142.24 91.44 0)
+			(effects
+				(font
+					(size 1.27 1.27)
+				)
+			)
+		)
+		(property "Footprint" ""
+			(at 142.24 96.52 0)
+			(effects
+				(font
+					(size 1.27 1.27)
+				)
+				(hide yes)
+			)
+		)
+		(property "Datasheet" ""
+			(at 142.24 96.52 0)
+			(effects
+				(font
+					(size 1.27 1.27)
+				)
+				(hide yes)
+			)
+		)
+		(property "Description" "Power symbol creates a global label with name \"+5V\""
+			(at 142.24 96.52 0)
+			(effects
+				(font
+					(size 1.27 1.27)
+				)
+				(hide yes)
+			)
+		)
+		(pin "1"
+		)
+		(instances
+			(project ""
+				(path "/2955ee96-3683-4cf6-bfa3-83b5e4980920/a9671bca-726d-4ae7-8d5c-45bb39bedd56"
+					(reference "#PWR027")
+					(unit 1)
+				)
+			)
 		)
 	)
@@
 			)
 		)
-		(property "Footprint" ""
+		(property "Footprint" "Capacitor_THT:CP_Radial_D5.0mm_P2.50mm"
 			(at 136.8552 104.14 0)
 			(effects
@@
 		)
 		(property "Description" "Polarized capacitor"
+			(at 135.89 100.33 0)
+			(effects
+				(font
+					(size 1.27 1.27)
+				)
+				(hide yes)
+			)
+		)
+		(property "amazon link" ""
 			(at 135.89 100.33 0)
 			(effects
@@
 			)
 		)
-		(property "Footprint" ""
+		(property "Footprint" "Resistor_SMD:R_0603_1608Metric_Pad0.98x0.95mm_HandSolder"
 			(at 120.3452 104.14 0)
 			(effects
@@
 		)
 		(property "Description" "Unpolarized capacitor"
+			(at 119.38 100.33 0)
+			(effects
+				(font
+					(size 1.27 1.27)
+				)
+				(hide yes)
+			)
+		)
+		(property "amazon link" ""
 			(at 119.38 100.33 0)
 			(effects
@@
 			)
 		)
-		(property "Footprint" ""
+		(property "Footprint" "Capacitor_THT:CP_Radial_D5.0mm_P2.50mm"
 			(at 181.3052 104.14 0)
 			(effects
@@
 		)
 		(property "Description" "Polarized capacitor"
+			(at 180.34 100.33 0)
+			(effects
+				(font
+					(size 1.27 1.27)
+				)
+				(hide yes)
+			)
+		)
+		(property "amazon link" ""
 			(at 180.34 100.33 0)
 			(effects
@@
 			)
 		)
-		(property "Footprint" ""
+		(property "Footprint" "Resistor_SMD:R_0603_1608Metric_Pad0.98x0.95mm_HandSolder"
 			(at 164.7952 104.14 0)
 			(effects
@@
 		)
 		(property "Description" "Unpolarized capacitor"
+			(at 163.83 100.33 0)
+			(effects
+				(font
+					(size 1.27 1.27)
+				)
+				(hide yes)
+			)
+		)
+		(property "amazon link" ""
 			(at 163.83 100.33 0)
 			(effects
@@
 			)
 		)
+		(property "amazon link" ""
+			(at 152.4 96.52 0)
+			(effects
+				(font
+					(size 1.27 1.27)
+				)
+				(hide yes)
+			)
+		)
 		(pin "3"
 		)
@@
 			)
 		)
-		(property "Footprint" ""
+		(property "Footprint" "TerminalBlock_Phoenix:TerminalBlock_Phoenix_MKDS-1,5-2_1x02_P5.00mm_Horizontal"
 			(at 99.06 99.06 0)
 			(effects
@@
 			(at 99.06 99.06 0)
 			(effects
+				(font
+					(size 1.27 1.27)
+				)
+				(hide yes)
+			)
+		)
+		(property "amazon link" "https://www.amazon.com/QSYZAIL-Screw-Terminal-Circuit-Connector/dp/B0G4MYNHBC/132-4224079-3597343"
+			(at 99.06 99.06 0)
+			(effects

Commit message: finishing the bom and adding the jlc number of the parts
Parts:
- C1, C3: jlc part # (none) -> C1591
- C2, C4: jlc part # (none) -> C216288
- J1: jlc part # (none) -> C3703
- U1: amazon link (none) -> https://www.amazon.com/Tegg-AMS1117-3-3V-Voltage-Regulator-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; jlc part # (none) -> C6186
Changed lines of the file:
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@@
+			)
+		)
+		(property "jlc part #" "C216288"
+			(at 135.89 100.33 0)
+			(effects
+				(font
+					(size 1.27 1.27)
+				)
+				(hide yes)
 			)
 		)
@@
 			)
 		)
+		(property "jlc part #" "C1591"
+			(at 119.38 100.33 0)
+			(effects
+				(font
+					(size 1.27 1.27)
+				)
+				(hide yes)
+			)
+		)
 		(pin "2"
 		)
@@
 			)
 		)
+		(property "jlc part #" "C216288"
+			(at 180.34 100.33 0)
+			(effects
+				(font
+					(size 1.27 1.27)
+				)
+				(hide yes)
+			)
+		)
 		(pin "2"
 		)
@@
 			)
 		)
+		(property "jlc part #" "C1591"
+			(at 163.83 100.33 0)
+			(effects
+				(font
+					(size 1.27 1.27)
+				)
+				(hide yes)
+			)
+		)
 		(pin "2"
 		)
@@
 			)
 		)
-		(property "amazon link" ""
+		(property "amazon link" "https://www.amazon.com/Tegg-AMS1117-3-3V-Voltage-Regulator-AMS1117/dp/B07X75XXYL?"
+			(at 152.4 96.52 0)
+			(effects
+				(font
+					(size 1.27 1.27)
+				)
+				(hide yes)
+			)
+		)
+		(property "jlc part #" "C6186"
 			(at 152.4 96.52 0)
 			(effects
@@
 			(at 99.06 99.06 0)
 			(effects
+				(font
+					(size 1.27 1.27)
+				)
+				(hide yes)
+			)
+		)
+		(property "jlc part #" "C3703"
+			(at 99.06 99.06 0)
+			(effects

Commit message: redesigning the power input
Parts:
- removed J1: Screw_Terminal_01x02, TerminalBlock_Phoenix:TerminalBlock_Phoenix_MKDS-1,5-2_1x02_P5.00mm_Horizontal, symbol Connector:Screw_Terminal_01x02
- added J1: USB_C_Receptacle_PowerOnly_6P, Connector_USB:USB_C_Receptacle_GCT_USB4125-xx-x_6P_TopMnt_Horizontal, symbol Connector:USB_C_Receptacle_PowerOnly_6P
- added R6, R7: 5,1k, symbol Device:R
Connections:
- net +5V: now also J1.A9 (VBUS), J1.B9 (VBUS)
- net GND: now also J1.A12 (GND), J1.B12 (GND), J1.S1 (SHIELD), R6.2, R7.2
- new net: J1.A5 (CC1), R6.1
- new net: J1.B5 (CC2), R7.1

Commit message: adding the components
Parts:
- J1: jlc part # (none) -> C456012
- R6, R7: footprint (none) -> Resistor_SMD:R_0603_1608Metric_Pad0.98x0.95mm_HandSolder; jlc part # (none) -> C177348
Changed lines of the file:
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@@
 			)
 		)
-		(property "Footprint" ""
+		(property "Footprint" "Resistor_SMD:R_0603_1608Metric_Pad0.98x0.95mm_HandSolder"
 			(at 73.66 90.678 90)
 			(effects
@@
 		(property "Description" "Resistor"
 			(at 73.66 88.9 0)
+			(effects
+				(font
+					(size 1.27 1.27)
+				)
+				(hide yes)
+			)
+		)
+		(property "jlc part #" "C177348"
+			(at 73.66 88.9 90)
 			(effects
 				(font
@@
 			)
 		)
-		(property "Footprint" ""
+		(property "Footprint" "Resistor_SMD:R_0603_1608Metric_Pad0.98x0.95mm_HandSolder"
 			(at 73.66 89.662 90)
 			(effects
@@
 		(property "Description" "Resistor"
 			(at 73.66 91.44 0)
+			(effects
+				(font
+					(size 1.27 1.27)
+				)
+				(hide yes)
+			)
+		)
+		(property "jlc part #" "C177348"
+			(at 73.66 91.44 90)
 			(effects
 				(font
@@
 			(at 54.61 83.82 0)
 			(effects
+				(font
+					(size 1.27 1.27)
+				)
+				(hide yes)
+			)
+		)
+		(property "jlc part #" "C456012"
+			(at 54.61 83.82 0)
+			(effects

Commit message: Finding parts and folishing the pcb
Parts:
- C2, C4: footprint Capacitor_THT:CP_Radial_D5.0mm_P2.50mm -> Capacitor_THT:CP_Radial_D5.0mm_P2.00mm
Changed lines of the file:
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@@
 			)
 		)
-		(property "Footprint" "Capacitor_THT:CP_Radial_D5.0mm_P2.50mm"
+		(property "Footprint" "Capacitor_THT:CP_Radial_D5.0mm_P2.00mm"
 			(at 136.8552 104.14 0)
 			(effects
@@
 			)
 		)
-		(property "Footprint" "Capacitor_THT:CP_Radial_D5.0mm_P2.50mm"
+		(property "Footprint" "Capacitor_THT:CP_Radial_D5.0mm_P2.00mm"
 			(at 181.3052 104.14 0)
 			(effects

Commit message: separating the pcb components from the other BOM
Parts:
- R6, R7: jlc part # C177348 -> C2907044
- U1: amazon link https://www.amazon.com/Tegg-AMS1117-3-3V-Voltage-Regulator-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 -> (none)
Changed lines of the file:
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@@
 			)
 		)
-		(property "jlc part #" "C177348"
+		(property "jlc part #" "C2907044"
 			(at 73.66 88.9 90)
 			(effects
@@
 			)
 		)
-		(property "jlc part #" "C177348"
+		(property "jlc part #" "C2907044"
 			(at 73.66 91.44 90)
 			(effects
@@
 			)
 		)
-		(property "amazon link" ""
-			(at 135.89 100.33 0)
-			(effects
-				(font
-					(size 1.27 1.27)
-				)
-				(hide yes)
-			)
-		)
 		(property "jlc part #" "C216288"
 			(at 135.89 100.33 0)
@@
 			)
 		)
-		(property "amazon link" ""
-			(at 119.38 100.33 0)
-			(effects
-				(font
-					(size 1.27 1.27)
-				)
-				(hide yes)
-			)
-		)
 		(property "jlc part #" "C1591"
 			(at 119.38 100.33 0)
@@
 			)
 		)
-		(property "amazon link" ""
-			(at 180.34 100.33 0)
-			(effects
-				(font
-					(size 1.27 1.27)
-				)
-				(hide yes)
-			)
-		)
 		(property "jlc part #" "C216288"
 			(at 180.34 100.33 0)
@@
 			)
 		)
-		(property "amazon link" ""
-			(at 163.83 100.33 0)
-			(effects
-				(font
-					(size 1.27 1.27)
-				)
-				(hide yes)
-			)
-		)
 		(property "jlc part #" "C1591"
 			(at 163.83 100.33 0)
@@
 			(at 152.4 96.52 0)
 			(effects
-				(font
-					(size 1.27 1.27)
-				)
-				(hide yes)
-			)
-		)
-		(property "amazon link" "https://www.amazon.com/Tegg-AMS1117-3-3V-Voltage-Regulator-AMS1117/dp/B07X75XXYL?"
-			(at 152.4 96.52 0)
-			(effects
