File: pcb/untitled.kicad_sch (KiCad schematic)
At the start: 1 part, among them J8 Screw_Terminal_01x07

Commit message: separating the pcb components from the other BOM
Parts:
- J8: amazon link https://www.amazon.com/LuoQiuFa10-7-Pin-5-08mm-Female-Termi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 -> (none)
Changed lines of the file:
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@@
-			)
-		)
-		(property "amazon link" "https://www.amazon.com/LuoQiuFa10-7-Pin-5-08mm-Female-Terminal/dp/B093DNFMLK?crid=10T3KHCJJYQ9W&"
-			(at 132.08 104.14 0)
-			(effects
-				(font
-					(size 1.27 1.27)
-				)
-				(hide yes)
 			)
 		)
