File: pcb/untitled.kicad_sch (KiCad schematic)
At the start: 1 part, among them J8 Screw_Terminal_01x07

Commit message: redesigning the circuit of the rellay and starting to adjust the footprints
Parts:
- J8: amazon link (none) -> https://www.amazon.com/LuoQiuFa10-7-Pin-5-08mm-Female-Termi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
Changed lines of the file:
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@@
+			)
+		)
+		(property "amazon link" "https://www.amazon.com/LuoQiuFa10-7-Pin-5-08mm-Female-Terminal/dp/B093DNFMLK?crid=10T3KHCJJYQ9W&"
+			(at 132.08 104.14 0)
+			(effects
+				(font
+					(size 1.27 1.27)
+				)
+				(hide yes)
 			)
 		)

Commit message: finishing the bom and adding the jlc number of the parts
Parts:
- J8: footprint (none) -> TerminalBlock_Phoenix:TerminalBlock_Phoenix_MKDS-1,5-7_1x07_P5.00mm_Horizontal; jlc part # (none) -> C395855
Changed lines of the file:
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@@
 			)
 		)
-		(property "Footprint" ""
+		(property "Footprint" "TerminalBlock_Phoenix:TerminalBlock_Phoenix_MKDS-1,5-7_1x07_P5.00mm_Horizontal"
 			(at 132.08 104.14 0)
 			(effects
@@
 			(at 132.08 104.14 0)
 			(effects
+				(font
+					(size 1.27 1.27)
+				)
+				(hide yes)
+			)
+		)
+		(property "jlc part #" "C395855"
+			(at 132.08 104.14 0)
+			(effects

Commit message: Finishing the carrier board with the new usb-c modul
Parts:
- renumbered J8 to J6
Changed lines of the file:
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@@
 		(dnp no)
 		(fields_autoplaced yes)
-		(property "Reference" "J8"
+		(property "Reference" "J6"
 			(at 134.62 102.8699 0)
 			(show_name no)
@@
 			(project "pcb"
 				(path "/2955ee96-3683-4cf6-bfa3-83b5e4980920/e294b273-6e19-4b0a-9116-e4dd566db649"
-					(reference "J8")
+					(reference "J6")
 					(unit 1)
 				)
@@
 		(dnp no)
 		(fields_autoplaced yes)
-		(property "Reference" "#PWR015"
+		(property "Reference" "#PWR014"
 			(at 120.65 109.22 0)
 			(hide yes)
@@
 			(project "pcb"
 				(path "/2955ee96-3683-4cf6-bfa3-83b5e4980920/e294b273-6e19-4b0a-9116-e4dd566db649"
-					(reference "#PWR015")
+					(reference "#PWR014")
 					(unit 1)
 				)
@@
 		(dnp no)
 		(fields_autoplaced yes)
-		(property "Reference" "#PWR016"
+		(property "Reference" "#PWR015"
 			(at 130.81 111.76 0)
 			(hide yes)
@@
 			(project "pcb"
 				(path "/2955ee96-3683-4cf6-bfa3-83b5e4980920/e294b273-6e19-4b0a-9116-e4dd566db649"
-					(reference "#PWR016")
+					(reference "#PWR015")
 					(unit 1)
 				)
