File: pcb/Programing pins.kicad_sch (KiCad schematic)
At the start: 1 part, among them J2 Conn_01x04_Pin

Commit message: redesigning the circuit of the rellay and starting to adjust the footprints
Parts:
- J2: amazon link (none) -> https://www.amazon.com/QSYZAIL-Screw-Terminal-Circuit-Conne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
Changed lines of the file:
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@@
+			)
+		)
+		(property "amazon link" "https://www.amazon.com/QSYZAIL-Screw-Terminal-Circuit-Connector/dp/B0G4MYNHBC/132-4224079-3597343"
+			(at 143.51 100.33 0)
+			(effects
+				(font
+					(size 1.27 1.27)
+				)
+				(hide yes)
 			)
 		)

Commit message: finishing the bom and adding the jlc number of the parts
Parts:
- J2: jlc part # (none) -> C37208
Changed lines of the file:
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@@
+			)
+		)
+		(property "jlc part #" "C37208"
+			(at 143.51 100.33 0)
+			(effects
+				(font
+					(size 1.27 1.27)
+				)
+				(hide yes)
 			)
 		)

Commit message: fixing the layout
Parts:
- J2: amazon link https://www.amazon.com/QSYZAIL-Screw-Terminal-Circuit-Conne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 -> (none)
Changed lines of the file:
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@@
 			)
 		)
-		(property "amazon link" "https://www.amazon.com/QSYZAIL-Screw-Terminal-Circuit-Connector/dp/B0G4MYNHBC/132-4224079-3597343"
+		(property "amazon link" ""
 			(at 143.51 100.33 0)
 			(effects

Commit message: Finishing the carrier board with the new usb-c modul
Parts:
- renumbered J2 to J8
Changed lines of the file:
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@@
 		(dnp no)
 		(fields_autoplaced yes)
-		(property "Reference" "#PWR06"
+		(property "Reference" "#PWR020"
 			(at 132.08 102.87 0)
 			(hide yes)
@@
 			(project "pcb"
 				(path "/2955ee96-3683-4cf6-bfa3-83b5e4980920/37c797a8-b815-44a0-8595-c386576311d4"
-					(reference "#PWR06")
+					(reference "#PWR020")
 					(unit 1)
 				)
@@
 		(in_pos_files yes)
 		(dnp no)
-		(property "Reference" "J2"
+		(property "Reference" "J8"
 			(at 136.652 89.662 0)
 			(show_name no)
@@
 			(project "pcb"
 				(path "/2955ee96-3683-4cf6-bfa3-83b5e4980920/37c797a8-b815-44a0-8595-c386576311d4"
-					(reference "J2")
+					(reference "J8")
 					(unit 1)
 				)
@@
 		(in_pos_files yes)
 		(dnp no)
-		(property "Reference" "#PWR05"
+		(property "Reference" "#PWR019"
 			(at 142.24 95.25 0)
 			(hide yes)
@@
 			(project "pcb"
 				(path "/2955ee96-3683-4cf6-bfa3-83b5e4980920/37c797a8-b815-44a0-8595-c386576311d4"
-					(reference "#PWR05")
+					(reference "#PWR019")
 					(unit 1)
 				)
