File: pcb/pump_control.kicad_sch (KiCad schematic)
At the start: 5 parts, among them J6 Screw_Terminal_01x02, K1 SANYOU_SRD_Form_A, Q1 2N2222A

Commit message: Finishing the carrier board with the new usb-c modul
Parts:
- renumbered J6 to J9, Q1 to Q2, R5 to R3
Changed lines of the file:
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@@
 		(in_pos_files yes)
 		(dnp no)
-		(property "Reference" "Q1"
+		(property "Reference" "Q2"
 			(at 142.24 110.4899 0)
 			(show_name no)
@@
 			(project "pcb"
 				(path "/2955ee96-3683-4cf6-bfa3-83b5e4980920/1e49f6cd-b5ca-46ba-8432-16205c4ff970"
-					(reference "Q1")
+					(reference "Q2")
 					(unit 1)
 				)
@@
 		(dnp no)
 		(fields_autoplaced yes)
-		(property "Reference" "J6"
+		(property "Reference" "J9"
 			(at 162.56 93.9799 0)
 			(show_name no)
@@
 			(project "pcb"
 				(path "/2955ee96-3683-4cf6-bfa3-83b5e4980920/1e49f6cd-b5ca-46ba-8432-16205c4ff970"
-					(reference "J6")
+					(reference "J9")
 					(unit 1)
 				)
@@
 		(dnp no)
 		(fields_autoplaced yes)
-		(property "Reference" "#PWR028"
+		(property "Reference" "#PWR021"
 			(at 139.7 74.93 0)
 			(hide yes)
@@
 			(project "pcb"
 				(path "/2955ee96-3683-4cf6-bfa3-83b5e4980920/1e49f6cd-b5ca-46ba-8432-16205c4ff970"
-					(reference "#PWR028")
+					(reference "#PWR021")
 					(unit 1)
 				)
@@
 		(dnp no)
 		(fields_autoplaced yes)
-		(property "Reference" "#PWR013"
+		(property "Reference" "#PWR022"
 			(at 139.7 123.19 0)
 			(hide yes)
@@
 			(project "pcb"
 				(path "/2955ee96-3683-4cf6-bfa3-83b5e4980920/1e49f6cd-b5ca-46ba-8432-16205c4ff970"
-					(reference "#PWR013")
+					(reference "#PWR022")
 					(unit 1)
 				)
@@
 		(dnp no)
 		(fields_autoplaced yes)
-		(property "Reference" "R5"
+		(property "Reference" "R3"
 			(at 124.46 105.41 90)
 			(show_name no)
@@
 			(project "pcb"
 				(path "/2955ee96-3683-4cf6-bfa3-83b5e4980920/1e49f6cd-b5ca-46ba-8432-16205c4ff970"
-					(reference "R5")
+					(reference "R3")
 					(unit 1)
 				)
