File: pcb/mainboard/Sensor inputs.kicad_sch (KiCad schematic)
At the start: 4 parts, among them J2 Screw_Terminal_01x04, J3 Screw_Terminal_01x02, J4 Screw_Terminal_01x03, J5 Screw_Terminal_01x03

Commit message: fixing some issues
Connections:
- net +3.3V: no longer J3.2 (Pin_2)
- net GND: now also J3.2 (Pin_2)
Changed lines of the file:
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@@
 	)
 	(symbol
-		(lib_id "power:+3.3V")
-		(at 147.32 127 270)
+		(lib_id "power:GND")
+		(at 147.32 127 90)
 		(unit 1)
 		(body_style 1)
@@
 		(fields_autoplaced yes)
 		(property "Reference" "#PWR08"
-			(at 143.51 127 0)
+			(at 153.67 127 0)
 			(hide yes)
 			(show_name no)
@@
 			)
 		)
-		(property "Value" "+3.3V"
+		(property "Value" "GND"
 			(at 151.13 126.9999 90)
 			(show_name no)
@@
 					(size 1.27 1.27)
 				)
-				(justify left)
+				(justify right)
 			)
 		)
@@
 			)
 		)
-		(property "Description" "Power symbol creates a global label with name \"+3.3V\""
+		(property "Description" "Power symbol creates a global label with name \"GND\" , ground"
 			(at 147.32 127 0)
 			(hide yes)
